File: ble_door_sensor.kicad_pcb (KiCad board)
At the start: 2 copper layers, 25.4 x 38.1 mm, 29 parts, among them IC1 MLPF-NRG-01D3, IC2 TCS40DPR,LF, U1 STM32WB09KEVx, Y1 NX2016SA-32M-EXS00A-CS06465, Y2 32.768KHz

Commit message: Rev B: VDDA_VCAP cap + battery divider + JST-MX 4P connector
PCB Rev B (title block "1.1/B", comment "Added: GPIOs connector.").
Boards ordered from fab. Folds in everything that was hand-reworked
on Rev A plus a new expansion connector for future modularity work.

Schematic + PCB changes vs Rev A:

1. **VDDA_VCAP decoupling cap** (0.22 µF) on STM32WB09KEVx pin 28.
   Rev A was missing this — caused HCI Hardware_Code 0x01 on every
   advert TX until hand-soldered. Now built into the layout.

2. **External battery-monitor divider**: R1 = 1 MΩ from cell+ →
   midpoint, R2 = 1 MΩ midpoint → GND, C1 = 1 µF X7R as a reservoir
   cap on the R2 side (NOT in series). Midpoint routed to PB1 =
   ADC1_VINP1. Quiescent ~1.5 µA. Replaces the Rev A hand-solder.

   Two bring-up gotchas were discovered with this circuit and are
   documented in the firmware repo:
     - PB3 (the original choice per all WB09 NUCLEO ADC examples)
       has a legacy JTDO default ~40 kΩ pull-up that can't be cleared
       from software. PB1 = VINP1 is the working alternative.
     - The WB0 ADC's sample-and-hold pulls ~7 nC per conversion;
       10 nF reservoir cap is too small (causes ~700 mV droop).
       1 µF X7R is the working value.

3. **JST-MX 4P expansion connector** on PA8 / PA9 / PA10 / PA11.
   Adds 4 GPIO lines to an external connector for future modular
   expansion (planned: motherboard + sensor-extension architecture
   where this connector is the m/b-side socket).

README:
- Replaces hero-image placeholder with side-A + side-B KiCad
  renders embedded via raw.githubusercontent URLs from sensorkit.

Tagged pcb-rev-b on this commit; pcb-rev-a remains as the
"as-fabricated original" reference.

Co-Authored-By: Claude Opus 4.7 (1M context) <noreply@anthropic.com>
Parts:
- added C13: 0.1uF, Capacitor_SMD:C_0603_1608Metric, F.Cu at (104.3, 61.2)
- added J1: Conn_01x04_Pin, KiCad:JST_MX_4P-1_25, F.Cu at (99.1, 80.1)
- added R3: 1M, Resistor_SMD:R_0402_1005Metric, F.Cu at (102.1, 61.5)
- R2: value 10K -> 1M
- moved R2 10.3 mm to (103.5, 64.6)
- moved C12 5.65 mm to (106.9, 59.6)
- moved IC2 4.83 mm to (97.8, 73.5), turned to 90 degrees
- moved R1 4.37 mm to (97.2, 66.5)
- moved D1 3.74 mm to (97.7, 68.7), turned to 90 degrees
- moved C1 0.23 mm to (109.7, 77.0)
- moved Y2 0.08 mm to (113.8, 71.8), turned to 90 degrees
Connections:
- C2 pad 1: GND -> Net-(U1-PB12)
- C2 pad 2: Net-(U1-PB12) -> GND
- R2 pad 2: Net-(U1-RSTN) -> Net-(U1-PB1)
- U1 pad 10: unconnected-(U1-PA9-Pad10) -> Net-(J1-Pin_3)
- U1 pad 11: unconnected-(U1-PA10-Pad11) -> Net-(J1-Pin_2)
- U1 pad 12: unconnected-(U1-PA11-Pad12) -> Net-(J1-Pin_1)
- U1 pad 3: unconnected-(U1-PB1-Pad3) -> Net-(U1-PB1)
- U1 pad 9: unconnected-(U1-PA8-Pad9) -> Net-(J1-Pin_4)
- Y2 pad 1: Net-(U1-PB12) -> Net-(U1-PB13)
- Y2 pad 2: Net-(U1-PB13) -> Net-(U1-PB12)
Routing:
- net Net-(U1-PB1): track 0.00 -> 16.8 mm
- net Net-(J1-Pin_4): track 0.00 -> 12.7 mm
- net GND: track 10.7 -> 23.2 mm, vias 45 -> 50
- net Net-(J1-Pin_3): track 0.00 -> 12.1 mm
- net Net-(J1-Pin_2): track 0.00 -> 11.5 mm
- net Net-(J1-Pin_1): track 0.00 -> 10.8 mm
- net Net-(U1-RSTN): track 21.3 -> 15.0 mm
- net Net-(IC2-VOUT): track 12.8 -> 7.98 mm
- net Net-(D1-K): track 8.53 -> 11.1 mm
- net +3V3: track 101.5 -> 103.0 mm
- net /SWCLK: track 21.4 -> 22.6 mm
